File: kicad/Attiny13ServoTester.kicad_pcb (KiCad board)
At the start: 2 copper layers, 13 parts, among them J1 POWER, J2 SERVO, J3 SERVO, SW1 SW_Push, U1 ATtiny13A-SSU, U2 AMS1117-3.3

Commit message: finishing project
Parts:
- added J4: PROG_SCK, Connector_Pin:Pin_D0.7mm_L6.5mm_W1.8mm_FlatFork, F.Cu at (151.3, 100.8)
- added J5: PROG_MOSI, Connector_Pin:Pin_D0.7mm_L6.5mm_W1.8mm_FlatFork, F.Cu at (150.7, 104.6)
- added J6: PROG_RESET, Connector_Pin:Pin_D0.7mm_L6.5mm_W1.8mm_FlatFork, F.Cu at (141.1, 100.3)
- added J7: PROG_MISO, Connector_Pin:Pin_D0.7mm_L6.5mm_W1.8mm_FlatFork, F.Cu at (153.8, 102.1)
- added R3: 1k, Resistor_SMD:R_0603_1608Metric_Pad1.05x0.95mm_HandSolder, F.Cu at (165.1, 91.2)
- moved J2 114.8 mm to (161.2, 81.8)
- moved SW1 114.8 mm to (130.2, 97.8)
- moved J3 114.8 mm to (164.8, 81.8)
- moved R2 114.8 mm to (155.6, 84.2)
- moved C1 114.8 mm to (162.5, 101.8)
- moved C2 114.8 mm to (158.7, 101.8)
- moved D1 114.8 mm to (139.1, 81.3)
- moved D2 114.8 mm to (154.3, 81.3)
- moved J1 114.8 mm to (130.2, 82.5)
- moved RV1 114.8 mm to (149.2, 96.5)
- moved U1 114.8 mm to (146.7, 101.6)
- moved U2 114.8 mm to (160.7, 95.2)
- moved R1 114.8 mm to (137.8, 84.7)
Connections:
- U1 pad 5: Net-(J2-Pad3) -> Net-(J5-Pad1)
Routing:
- net Net-(J5-Pad1): track 0.00 -> 29.5 mm
- net Net-(J2-Pad3): track 35.5 -> 7.18 mm
- net Net-(J7-Pad1): track 14.6 -> 19.0 mm
- net Net-(J6-Pad1): track 0.00 -> 3.20 mm
- net Net-(J4-Pad1): track 5.83 -> 7.75 mm
- net Net-(C2-Pad2): track 19.3 -> 21.1 mm
